File: continuity.sch (KiCad schematic (older format))
At the start: 30 parts, among them J1 Conn_01x01_Female, J2 Conn_01x04_Female, J3 Conn_01x01_Female, Q1 BCP52, Q2 BCP55, Q3 BCP55, U1 MCP 6V11T-EOT

Commit message: snap
Parts:
- removed J1: Conn_01x01_Female, MountingHole:MountingHole_4mm_Pad_Via, symbol Connector:Conn_01x01_Female
- removed J2: Conn_01x04_Female, continuity:KEYSTONE_1012, symbol Connector:Conn_01x04_Female
- added BAT1, GREEN2, LS2, PROBE1, RED2: Conn_01x02_Male, Connector_JST:JST_XH_B2B-XH-A_1x02_P2.50mm_Vertical, symbol Connector:Conn_01x02_Male
- added FID1, FID2: Fiducial, Fiducial:Fiducial_Modern_CopperTop, symbol Mechanical:Fiducial
- added GREEN1: LED, LED_SMD:LED_PLCC-2, symbol Device:LED
- added H1, H2, H3, H4: MountingHole, MountingHole:MountingHole_3.2mm_M3, symbol Mechanical:MountingHole
- added J5: Buchse Rot, symbol Connector:Conn_01x01_Female
- added N3: LED Fassung, symbol Mechanical:Housing
- added NT1: Net-Tie_2, NetTie:NetTie-2_SMD_Pad0.5mm, symbol Device:Net-Tie_2
- added R14, R15: 240, Resistor_SMD:R_0603_1608Metric_Pad1.05x0.95mm_HandSolder, symbol Device:R
- added Ra1: 470, Resistor_SMD:R_1206_3216Metric_Pad1.42x1.75mm_HandSolder, symbol Device:R
- added TP1: VCC, TestPoint:TestPoint_THTPad_1.0x1.0mm_Drill0.5mm, symbol Connector:TestPoint_Flag
- added TP2: PROBE, TestPoint:TestPoint_THTPad_1.0x1.0mm_Drill0.5mm, symbol Connector:TestPoint_Flag
- added TP3: SENSE, TestPoint:TestPoint_THTPad_1.0x1.0mm_Drill0.5mm, symbol Connector:TestPoint_Flag
- added TP4: PROBE_uA, TestPoint:TestPoint_THTPad_1.0x1.0mm_Drill0.5mm, symbol Connector:TestPoint_Flag
- added TP5: VCC_SW, TestPoint:TestPoint_THTPad_1.0x1.0mm_Drill0.5mm, symbol Connector:TestPoint_Flag
- added TP6: KOMP_OUT, TestPoint:TestPoint_THTPad_1.0x1.0mm_Drill0.5mm, symbol Connector:TestPoint_Flag
- added TP7: OUT, TestPoint:TestPoint_THTPad_1.0x1.0mm_Drill0.5mm, symbol Connector:TestPoint_Flag
- added TP8: GND, TestPoint:TestPoint_THTPad_1.0x1.0mm_Drill0.5mm, symbol Connector:TestPoint_Flag
- J3: value Conn_01x01_Female -> Buchse Schwarz; footprint MountingHole:MountingHole_4mm_Pad_Via -> (none)
- LS1: footprint Buzzer_Beeper:Buzzer_CUI_CPT-9019S-SMT -> Buzzer_Beeper:Buzzer_15x7.5RM7.6
- N1: value Housing -> Testkabel
- N2: Vendor RND 455-00908 -> 1553CBKBAT
- R3: value 5k -> 4,7k
- Rb1: renamed from R1; value 240 -> 470; footprint Resistor_SMD:R_0805_2012Metric_Pad1.15x1.40mm_HandSolder -> Resistor_SMD:R_1206_3216Metric_Pad1.42x1.75mm_HandSolder; Vendor RND 0805 1 240 -> RND 155HP06 DD
- U1: symbol Amplifier_Operational:MCP6L91RT-EOT -> Amplifier_Operational:MCP6L91T-EOT
- renumbered D1 to RED1
Connections:
- net labels added: KOMP_OUT, Probe, Probe_uA
- wire segments 71 -> 102
Other:
- moved on the sheet: D3, LS1, N1, R2

Commit message: snap
Parts:
- LS1: Vendor VIS 3580 -> RND 430-00009
Connections:
- wire segments 102 -> 100
Changed lines of the file:
@@
 F 2 "Buzzer_Beeper:Buzzer_15x7.5RM7.6" H 7465 2650 50  0001 C CNN
 F 3 "~" H 7465 2650 50  0001 C CNN
-F 4 "VIS 3580" H 7500 2700 50  0001 C CNN "Vendor"
+F 4 "RND 430-00009" H 7500 2700 50  0001 C CNN "Vendor"
 	1    7500 2700
 	-1   0    0    -1
@@
 	8150 2700 8150 2800
 Wire Wire Line
-	8150 2700 8200 2700
-Wire Wire Line
 	7500 3100 7900 3100
 $Comp
@@
 Wire Wire Line
 	8150 2250 8150 2700
-Wire Wire Line
-	8150 2700 8200 2700
 Connection ~ 6300 2250
 Wire Wire Line
 	6300 2250 6300 2450
 Connection ~ 8150 2700
-Connection ~ 8200 2700
-Wire Wire Line
-	8200 2700 8450 2700
+Wire Wire Line
+	8150 2700 8450 2700
 $EndSCHEMATC
